Commit message: completed simulation darknet_ros+kcf down tracking

File: src/simulation/urdf/car/prius_a02.urdf (robot description, URDF)
Before this commit: robot prius, 13 links, 12 joints
Links:
- added link planding_place, mass 0.1; visual mesh filename=package://simulation/urdf/car/meshes/landing.dae scale=3 3 3
Joints:
- added joint landing_link_connection: type fixed, parent chassis, child planding_place, origin xyz=0.4 2.2 1.5 rpy=-1.57 0 0, axis 1 0 0
